Commit message: Re-arrange folders

File: models/diag_Y_positive_10_lifted/model.urdf (robot description, URDF)
Before this commit: robot Y_positive_10_lifted, 2 links, 1 joints
Links:
- removed link Y_positive_10_lifted__link
- added link diag_Y_positive_10_lifted__link, mass 10; collision mesh filename=package://pal_gazebo_worlds/models/diag_Y_positive_10_lifte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 scale=0.00999 0.00999 0.00999; visual mesh filename=package://pal_gazebo_worlds/models/diag_Y_positive_10_lifte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 scale=0.00999 0.00999 0.00999
Joints:
- joint fixed: child Y_positive_10_lifted__link -> diag_Y_positive_10_lifted__link

File: models/diag_Y_positive_10_lifted_size_30/model.urdf (robot description, URDF)
Before this commit: robot Y_positive_10_lifted, 2 links, 1 joints
Links:
- removed link Y_positive_10_lifted__link
- added link diag_Y_positive_10_lifted_size_30__link, mass 10; collision mesh filename=package://pal_gazebo_worlds/models/diag_Y_positive_10_lifte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 scale=0.00999 0.00999 0.00999; visual mesh filename=package://pal_gazebo_worlds/models/diag_Y_positive_10_lifte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 scale=0.00999 0.00999 0.00999
Joints:
- joint fixed: child Y_positive_10_lifted__link -> diag_Y_positive_10_lifted_size_30__link

File: models/diag_Y_positive_15_lifted/model.urdf (robot description, URDF)
Before this commit: robot Y_positive_10_lifted, 2 links, 1 joints
Links:
- removed link Y_positive_10_lifted__link
- added link diag_Y_positive_15_lifted__link, mass 10; collision mesh filename=package://pal_gazebo_worlds/models/diag_Y_positive_15_lifte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 scale=0.00999 0.00999 0.00999; visual mesh filename=package://pal_gazebo_worlds/models/diag_Y_positive_15_lifte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 scale=0.00999 0.00999 0.00999
Joints:
- joint fixed: child Y_positive_10_lifted__link -> diag_Y_positive_15_lifted__link

File: models/diag_Y_positive_15_lifted_size_30/model.urdf (robot description, URDF)
Before this commit: robot Y_positive_10_lifted, 2 links, 1 joints
Links:
- removed link Y_positive_10_lifted__link
- added link diag_Y_positive_15_lifted_size_30__link, mass 10; collision mesh filename=package://pal_gazebo_worlds/models/diag_Y_positive_15_lifte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 scale=0.00999 0.00999 0.00999; visual mesh filename=package://pal_gazebo_worlds/models/diag_Y_positive_15_lifte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 scale=0.00999 0.00999 0.00999
Joints:
- joint fixed: child Y_positive_10_lifted__link -> diag_Y_positive_15_lifted_size_30__link
